File: Custom Macropad/Custom Macropad.kicad_sch (KiCad schematic)
At the start: 25 parts, among them SW1 RotaryEncoder_Switch, SW10 SW_Push, SW11 SW_Push, SW12 SW_Push, SW17 RotaryEncoder_Switch, SW2 SW_Push, SW3 SW_Push, SW5 SW_Push, SW6 SW_Push, SW7 SW_Push, SW8 SW_Push, SW9 SW_Push, U1 MOUDLE-SEEEDUINO-XIAO

Commit message: Schematic V1
Parts:
- removed SW1: RotaryEncoder_Switch, symbol Device:RotaryEncoder_Switch
- added D13, D14, D15, D16: 1N4148, Diode_THT:D_DO-35_SOD27_P7.62mm_Horizontal, symbol Diode:1N4148
- added D17, D18, D19, D20, D21, D22, D23, D24, D25, D26, D27, D28, D29, D30, D31, D32: WS2812B, LED_SMD:LED_WS2812B_PLCC4_5.0x5.0mm_P3.2mm, symbol LED:WS2812B
- added SW1, SW13, SW14, SW15, SW4: SW_Push, symbol Switch:SW_Push
Connections:
- net EC12A is gone; now on net EC11A: SW17.A, U1.6 (PA9_A5_D5_SCL)
- net EC12B is gone; now on net EC11B: SW17.B, U1.7 (PB08_A6_D6_TX)
- net +5V: now also D17.1 (VDD), D18.1 (VDD), D19.1 (VDD), D20.1 (VDD), D21.1 (VDD), D22.1 (VDD), D23.1 (VDD), D24.1 (VDD), D25.1 (VDD), D26.1 (VDD), D27.1 (VDD), D28.1 (VDD), D29.1 (VDD), D30.1 (VDD), D31.1 (VDD), D32.1 (VDD)
- net COL0: now also SW1.2, SW4.2
- net COL1: now also SW13.2
- net COL2: now also SW14.2
- net COL3: now also SW15.2
- net EC11A: no longer U1.4 (PA11_A3_D3)
- net EC11B: no longer U1.5 (PA8_A4_D4_SDA)
- net GND: now also D17.3 (VSS), D18.3 (VSS), D19.3 (VSS), D20.3 (VSS), D21.3 (VSS), D22.3 (VSS), D23.3 (VSS), D24.3 (VSS), D25.3 (VSS), D26.3 (VSS), D27.3 (VSS), D28.3 (VSS), D29.3 (VSS), D30.3 (VSS), D31.3 (VSS), D32.3 (VSS)
- net at D1.2 (A): now also SW1.1
- new net: D25.2 (DOUT), D26.4 (DIN)
- new net: D24.2 (DOUT), D25.4 (DIN)
- new net: D15.2 (A), SW14.1
- new net: D13.2 (A), SW4.1
- new net: D31.2 (DOUT), D32.4 (DIN)
- new net: D30.2 (DOUT), D31.4 (DIN)
- new net: D20.2 (DOUT), D21.4 (DIN)
- new net: D19.2 (DOUT), D20.4 (DIN)
- new net: D26.2 (DOUT), D27.4 (DIN)
- new net: D16.2 (A), SW15.1
- new net: D22.2 (DOUT), D23.4 (DIN)
- new net: D21.2 (DOUT), D22.4 (DIN)
- new net: D29.2 (DOUT), D30.4 (DIN)
- new net: D28.2 (DOUT), D29.4 (DIN)
- new net: D18.2 (DOUT), D19.4 (DIN)
- new net: D17.2 (DOUT), D18.4 (DIN)
- new net: D23.2 (DOUT), D24.4 (DIN)
- new net: D27.2 (DOUT), D28.4 (DIN)
- new net: D14.2 (A), SW13.1
- new net LEDC: D17.4 (DIN), U1.5 (PA8_A4_D4_SDA)
- new net ROW3: D13.1 (K), D14.1 (K), D15.1 (K), D16.1 (K), U1.4 (PA11_A3_D3)
Other:
- moved on the sheet: D1, D10, D11, D12, D2, D3, D4, D5, D6, D7, D8, D9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

Commit message: Key pcb layout
Parts:
- D17, D18, D19, D20, D21, D22, D23, D24, D25, D26, D27, D28, D29, D30, D31, D32: footprint LED_SMD:LED_WS2812B_PLCC4_5.0x5.0mm_P3.2mm -> footprints:SK6812MINI-E_fixed
- SW1, SW10, SW11, SW12, SW13, SW14, SW15, SW2, SW3, SW4, SW5, SW6, SW7, SW8, SW9: footprint (none) -> Button_Switch_Keyboard:SW_Cherry_MX_1.00u_PCB
- SW17: footprint (none) -> Rotary_Encoder:RotaryEncoder_Alps_EC11E-Switch_Vertical_H20mm
- U1: footprint (none) -> footprints:XIAO-Generic-Hybrid-14P-2.54-21X17.8MM
Changed lines of the file:
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@@
 			)
 		)
-		(property "Footprint" "LED_SMD:LED_WS2812B_PLCC4_5.0x5.0mm_P3.2mm"
+		(property "Footprint" "footprints:SK6812MINI-E_fixed"
 			(at 58.42 157.48 0)
 			(effects
@@
 			)
 		)
-		(property "Footprint" ""
+		(property "Footprint" "Button_Switch_Keyboard:SW_Cherry_MX_1.00u_PCB"
 			(at 59.69 44.45 0)
 			(effects
@@
 			)
 		)
-		(property "Footprint" "LED_SMD:LED_WS2812B_PLCC4_5.0x5.0mm_P3.2mm"
+		(property "Footprint" "footprints:SK6812MINI-E_fixed"
 			(at 187.96 157.48 0)
 			(effects
@@
 			)
 		)
-		(property "Footprint" "LED_SMD:LED_WS2812B_PLCC4_5.0x5.0mm_P3.2mm"
+		(property "Footprint" "footprints:SK6812MINI-E_fixed"
 			(at 123.19 128.27 0)
 			(effects
@@
 			)
 		)
-		(property "Footprint" "LED_SMD:LED_WS2812B_PLCC4_5.0x5.0mm_P3.2mm"
+		(property "Footprint" "footprints:SK6812MINI-E_fixed"
 			(at 80.01 157.48 0)
 			(effects
@@
 			)
 		)
-		(property "Footprint" ""
+		(property "Footprint" "Rotary_Encoder:RotaryEncoder_Alps_EC11E-Switch_Vertical_H20mm"
 			(at 91.694 38.1 0)
 			(effects
@@
 		(pin "S1"
 		)
+		(pin "MP"
+		)
 		(instances
 			(project ""
@@
 			)
 		)
-		(property "Footprint" ""
+		(property "Footprint" "Button_Switch_Keyboard:SW_Cherry_MX_1.00u_PCB"
 			(at 44.45 44.45 0)
 			(effects
@@
 			)
 		)
-		(property "Footprint" "LED_SMD:LED_WS2812B_PLCC4_5.0x5.0mm_P3.2mm"
+		(property "Footprint" "footprints:SK6812MINI-E_fixed"
 			(at 167.64 128.27 0)
 			(effects
@@
 			)
 		)
-		(property "Footprint" "LED_SMD:LED_WS2812B_PLCC4_5.0x5.0mm_P3.2mm"
+		(property "Footprint" "footprints:SK6812MINI-E_fixed"
 			(at 210.82 157.48 0)
 			(effects
@@
 			)
 		)
-		(property "Footprint" "LED_SMD:LED_WS2812B_PLCC4_5.0x5.0mm_P3.2mm"
+		(property "Footprint" "footprints:SK6812MINI-E_fixed"
 			(at 146.05 157.48 0)
 			(effects
@@
 			)
 		)
-		(property "Footprint" "LED_SMD:LED_WS2812B_PLCC4_5.0x5.0mm_P3.2mm"
+		(property "Footprint" "footprints:SK6812MINI-E_fixed"
 			(at 80.01 128.27 0)
 			(effects
@@
 			)
 		)
-		(property "Footprint" ""
+		(property "Footprint" "Button_Switch_Keyboard:SW_Cherry_MX_1.00u_PCB"
 			(at 59.69 78.74 0)
 			(effects
@@
 			)
 		)
-		(property "Footprint" ""
+		(property "Footprint" "Button_Switch_Keyboard:SW_Cherry_MX_1.00u_PCB"
 			(at 44.45 62.23 0)
 			(effects
@@
 			)
 		)
-		(property "Footprint" ""
+		(property "Footprint" "Button_Switch_Keyboard:SW_Cherry_MX_1.00u_PCB"
 			(at 90.17 95.25 0)
 			(effects
@@
 			)
 		)
-		(property "Footprint" "LED_SMD:LED_WS2812B_PLCC4_5.0x5.0mm_P3.2mm"
+		(property "Footprint" "footprints:SK6812MINI-E_fixed"
 			(at 187.96 128.27 0)
 			(effects
@@
 			)
 		)
-		(property "Footprint" "LED_SMD:LED_WS2812B_PLCC4_5.0x5.0mm_P3.2mm"
+		(property "Footprint" "footprints:SK6812MINI-E_fixed"
 			(at 100.33 157.48 0)
 			(effects
@@
 			)
 		)
-		(property "Footprint" "LED_SMD:LED_WS2812B_PLCC4_5.0x5.0mm_P3.2mm"
+		(property "Footprint" "footprints:SK6812MINI-E_fixed"
 			(at 123.19 157.48 0)
 			(effects
@@
 			)
 		)
-		(property "Footprint" "LED_SMD:LED_WS2812B_PLCC4_5.0x5.0mm_P3.2mm"
+		(property "Footprint" "footprints:SK6812MINI-E_fixed"
 			(at 100.33 128.27 0)
 			(effects
@@
 			)
 		)
-		(property "Footprint" "LED_SMD:LED_WS2812B_PLCC4_5.0x5.0mm_P3.2mm"
+		(property "Footprint" "footprints:SK6812MINI-E_fixed"
 			(at 167.64 157.48 0)
 			(effects
@@
 			)
 		)
-		(property "Footprint" ""
+		(property "Footprint" "Button_Switch_Keyboard:SW_Cherry_MX_1.00u_PCB"
 			(at 44.45 78.74 0)
 			(effects
@@
 			)
 		)
-		(property "Footprint" ""
+		(property "Footprint" "Button_Switch_Keyboard:SW_Cherry_MX_1.00u_PCB"
 			(at 74.93 78.74 0)
 			(effects
@@
 			)
 		)
-		(property "Footprint" "LED_SMD:LED_WS2812B_PLCC4_5.0x5.0mm_P3.2mm"
+		(property "Footprint" "footprints:SK6812MINI-E_fixed"
 			(at 210.82 128.27 0)
 			(effects
@@
 			)
 		)
-		(property "Footprint" "LED_SMD:LED_WS2812B_PLCC4_5.0x5.0mm_P3.2mm"
+		(property "Footprint" "footprints:SK6812MINI-E_fixed"
 			(at 58.42 128.27 0)
 			(effects
@@
 			)
 		)
-		(property "Footprint" "LED_SMD:LED_WS2812B_PLCC4_5.0x5.0mm_P3.2mm"
+		(property "Footprint" "footprints:SK6812MINI-E_fixed"
 			(at 146.05 128.27 0)
 			(effects
@@
 			)
 		)
-		(property "Footprint" ""
+		(property "Footprint" "Button_Switch_Keyboard:SW_Cherry_MX_1.00u_PCB"
 			(at 74.93 95.25 0)
 			(effects
@@
 			)
 		)
-		(property "Footprint" ""
+		(property "Footprint" "Button_Switch_Keyboard:SW_Cherry_MX_1.00u_PCB"
 			(at 59.69 62.23 0)
 			(effects
@@
 			)
 		)
-		(property "Footprint" ""
+		(property "Footprint" "Button_Switch_Keyboard:SW_Cherry_MX_1.00u_PCB"
 			(at 59.69 95.25 0)
 			(effects
@@
 			)
 		)
-		(property "Footprint" ""
+		(property "Footprint" "Button_Switch_Keyboard:SW_Cherry_MX_1.00u_PCB"
 			(at 90.17 78.74 0)
 			(effects
@@
 			)
 		)
-		(property "Footprint" ""
+		(property "Footprint" "Button_Switch_Keyboard:SW_Cherry_MX_1.00u_PCB"
 			(at 44.45 95.25 0)
 			(effects
@@
 			)
 		)
-		(property "Footprint" ""
+		(property "Footprint" "footprints:XIAO-Generic-Hybrid-14P-2.54-21X17.8MM"
 			(at 140.97 63.5 0)
 			(effects
@@
 			)
 		)
-		(property "Footprint" ""
+		(property "Footprint" "Button_Switch_Keyboard:SW_Cherry_MX_1.00u_PCB"
 			(at 74.93 62.23 0)
 			(effects
@@
 			)
 		)
-		(property "Footprint" ""
+		(property "Footprint" "Button_Switch_Keyboard:SW_Cherry_MX_1.00u_PCB"
 			(at 74.93 44.45 0)
 			(effects
@@
 			)
 		)
-		(property "Footprint" ""
+		(property "Footprint" "Button_Switch_Keyboard:SW_Cherry_MX_1.00u_PCB"
 			(at 90.17 62.23 0)
 			(effects

Commit message: full pcb layout done w/o routing
Parts:
- renumbered SW4 to SW13, SW13 to SW14, SW14 to SW15, SW15 to SW16, SW17 to SW4
Changed lines of the file:
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@@
 		(dnp no)
 		(fields_autoplaced yes)
-		(property "Reference" "SW17"
-			(at 93.98 40.6399 90)
+		(property "Reference" "SW4"
+			(at 93.98 41.8464 90)
 			(effects
 				(font
@@
 		)
 		(property "Value" "RotaryEncoder_Switch"
-			(at 93.98 43.1799 90)
+			(at 93.98 44.3864 90)
 			(effects
 				(font
@@
 			(project ""
 				(path "/cac26fb3-9366-413f-8bbf-885ac1b417bf"
-					(reference "SW17")
+					(reference "SW4")
 					(unit 1)
 				)
@@
 		(dnp no)
 		(fields_autoplaced yes)
-		(property "Reference" "SW15"
+		(property "Reference" "SW16"
 			(at 90.17 92.71 0)
 			(effects
@@
 			(project "Custom Macropad"
 				(path "/cac26fb3-9366-413f-8bbf-885ac1b417bf"
-					(reference "SW15")
+					(reference "SW16")
 					(unit 1)
 				)
@@
 		(dnp no)
 		(fields_autoplaced yes)
-		(property "Reference" "SW14"
+		(property "Reference" "SW15"
 			(at 74.93 92.71 0)
 			(effects
@@
 			(project "Custom Macropad"
 				(path "/cac26fb3-9366-413f-8bbf-885ac1b417bf"
-					(reference "SW14")
+					(reference "SW15")
 					(unit 1)
 				)
@@
 		(dnp no)
 		(fields_autoplaced yes)
-		(property "Reference" "SW13"
+		(property "Reference" "SW14"
 			(at 59.69 92.71 0)
 			(effects
@@
 			(project "Custom Macropad"
 				(path "/cac26fb3-9366-413f-8bbf-885ac1b417bf"
-					(reference "SW13")
+					(reference "SW14")
 					(unit 1)
 				)
@@
 		(dnp no)
 		(fields_autoplaced yes)
-		(property "Reference" "SW4"
+		(property "Reference" "SW13"
 			(at 44.45 92.71 0)
 			(effects
@@
 			(project "Custom Macropad"
 				(path "/cac26fb3-9366-413f-8bbf-885ac1b417bf"
-					(reference "SW4")
-					(unit 1)
-				)
+					(reference "SW13")
+					(unit 1)
+				)

Commit message: Finished routing v1
Connections:
- net GND: now also SW4.MP (Shield)
Changed lines of the file:
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@@
 	(wire
 		(pts
+			(xy 87.63 46.99) (xy 87.63 49.53)
+		)
+		(stroke
+			(width 0)
+			(type default)
+		)
+	)
+	(wire
+		(pts
 			(xy 78.74 113.03) (xy 57.15 113.03)
 		)
@@
 					(unit 1)
 				)
+			)
+		)
+	)
+	(symbol
+		(lib_id "power:GND")
+		(at 87.63 49.53 0)
+		(unit 1)
+		(exclude_from_sim no)
+		(in_bom yes)
+		(on_board yes)
+		(dnp no)
+		(fields_autoplaced yes)
+		(property "Reference" "#PWR07"
+			(at 87.63 55.88 0)
+			(effects
+				(font
+					(size 1.27 1.27)
+				)
+				(hide yes)
+			)
+		)
+		(property "Value" "GND"
+			(at 87.63 54.61 0)
+			(effects
+				(font
+					(size 1.27 1.27)
+				)
+			)
+		)
+		(property "Footprint" ""
+			(at 87.63 49.53 0)
+			(effects
+				(font
+					(size 1.27 1.27)
+				)
+				(hide yes)
+			)
+		)
+		(property "Datasheet" ""
+			(at 87.63 49.53 0)
+			(effects
+				(font
+					(size 1.27 1.27)
+				)
+				(hide yes)
+			)
+		)
+		(property "Description" "Power symbol creates a global label with name \"GND\" , ground"
+			(at 87.63 49.53 0)
+			(effects
+				(font
+					(size 1.27 1.27)
+				)
+				(hide yes)
+			)
+		)
+		(pin "1"
+		)
+		(instances
+			(project ""
+				(path "/cac26fb3-9366-413f-8bbf-885ac1b417bf"
+					(reference "#PWR07")
+					(unit 1)
+				)
