File: Custom Macropad/Custom Macropad.kicad_pcb (KiCad board)
At the start: 2 copper layers, 3.6 x 3.3 mm, 49 parts, among them SW1 SW_Push, SW10 SW_Push, SW11 SW_Push, SW12 SW_Push, SW13 SW_Push, SW14 SW_Push, SW15 SW_Push, SW17 RotaryEncoder_Switch, SW2 SW_Push, SW3 SW_Push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

Commit message: full pcb layout done w/o routing
Parts:
- U1: moved to B.Cu
- moved D24 147.5 mm to (185.7, 96.8)
- moved D28 147.3 mm to (185.7, 115.9)
- moved D32 146.5 mm to (185.7, 134.9)
- moved D19 135.2 mm to (166.7, 77.8)
- moved D20 132.7 mm to (163.5, 66.7)
- moved D31 131.2 mm to (166.7, 134.9)
- moved D23 129.9 mm to (166.7, 96.8)
- moved D27 129.6 mm to (166.7, 115.9)
- moved D30 117.2 mm to (147.6, 134.9)
- moved D18 116.3 mm to (147.6, 77.8)
- moved D22 116.3 mm to (147.6, 96.8)
- moved D26 112.7 mm to (147.6, 115.9)
- moved D29 105.4 mm to (128.8, 135.1)
- moved D17 97.8 mm to (128.6, 77.8)
- moved D21 97.7 mm to (128.6, 96.8)
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- renumbered SW4 to SW13, SW13 to SW14, SW14 to SW15, SW15 to SW16, SW17 to SW4

Commit message: Finished routing v1
Parts:
- moved D25 57.2 mm to (185.7, 115.9)
- moved D28 57.2 mm to (128.6, 115.9)
- moved D17 36.7 mm to (163.5, 66.7)
- moved D20 36.7 mm to (128.6, 77.8)
- moved D18 19.1 mm to (166.7, 77.8)
- moved D19 19.1 mm to (147.6, 77.8)
- moved D26 19.1 mm to (166.7, 115.9)
- moved D27 19.1 mm to (147.6, 115.9)
- moved D2 11.4 mm to (145.3, 81.8), turned to 0 degrees
- moved D4 1.75 mm to (183.6, 81.4)
- moved D7 0.79 mm to (174.6, 95.9)
- moved D8 0.79 mm to (193.7, 95.9)
- moved D1 0.51 mm to (136.0, 76.8)
Connections:
- SW4 pad MP: unconnected-(SW4-Shield-PadMP) -> GND
Routing:
- net +5V: track 0.00 -> 377.9 mm, vias 0 -> 27
- net GND: track 0.00 -> 373.4 mm, vias 0 -> 21
- net ROW3: track 0.00 -> 144.0 mm
- net ROW2: track 0.00 -> 130.5 mm, vias 0 -> 5
- net COL3: track 0.00 -> 106.6 mm, vias 0 -> 1
- net ROW1: track 0.00 -> 105.5 mm, vias 0 -> 5
- net ROW0: track 0.00 -> 103.1 mm, vias 0 -> 6
- net COL2: track 0.00 -> 88.7 mm, vias 0 -> 2
- net COL0: track 0.00 -> 73.4 mm
- net COL1: track 0.00 -> 61.0 mm, vias 0 -> 1
- net Net-(D22-DOUT): track 0.00 -> 52.1 mm, vias 0 -> 4
- net Net-(D30-DOUT): track 0.00 -> 41.8 mm, vias 0 -> 2
- net Net-(D23-DOUT): track 0.00 -> 38.2 mm, vias 0 -> 2
- net Net-(D21-DOUT): track 0.00 -> 37.3 mm, vias 0 -> 2
- net Net-(D31-DOUT): track 0.00 -> 34.0 mm, vias 0 -> 2
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Other:
- board text added: "K"

Commit message: Final
Other:
- board size 3.6 x 3.3 mm -> 77.8 x 77.8 mm
Changed lines of the file:
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@@
 		)
+	)
+	(gr_rect
+		(start 118.26875 62.70625)
+		(end 196.05625 140.49375)
+		(stroke
+			(width 0.05)
+			(type default)
+		)
+		(fill no)
+		(layer "Edge.Cuts")
 	)
 	(gr_text "K"
@@
 	)
 	(segment
-		(start 126.365 99.441)
-		(end 125.984 99.441)
+		(start 125.984 99.441)
+		(end 132.207 99.441)
 		(width 0.254)
 		(layer "F.Cu")
@@
 		(width 0.254)
 		(layer "F.Cu")
-		(net 28)
-	)
-	(segment
-		(start 132.207 99.441)
-		(end 126.365 99.441)
-		(width 0.254)
-		(layer "F.Cu")

Commit message: Final v2
Other:
- board size 77.8 x 77.8 mm -> 79.4 x 79.4 mm
Changed lines of the file:
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@@
 	)
 	(gr_rect
-		(start 118.26875 62.70625)
-		(end 196.05625 140.49375)
+		(start 117.475 61.9125)
+		(end 196.85 141.2875)
 		(stroke
 			(width 0.05)
@@
 		)
 	)
+	(dimension
+		(type orthogonal)
+		(layer "Edge.Cuts")
+		(pts
+			(xy 196.85 61.9125) (xy 196.85 141.2875)
+		)
+		(height 23.01875)
+		(orientation 1)
+		(format
+			(prefix "")
+			(suffix "")
+			(units 3)
+			(units_format 0)
+			(precision 4)
+			(suppress_zeroes yes)
+		)
+		(style
+			(thickness 0.05)
+			(arrow_length 1.27)
+			(text_position_mode 0)
+			(arrow_direction outward)
+			(extension_height 0.58642)
+			(extension_offset 0.5)
+			(keep_text_aligned yes)
+		)
+		(gr_text "79.375"
+			(at 218.71875 101.6 90)
+			(layer "Edge.Cuts")
+			(effects
+				(font
+					(size 1 1)
+					(thickness 0.15)
+				)
+			)
+		)
+	)
